File: ATX-PSU-ProtoHAT.kicad_sch (KiCad schematic)
At the start: 19 parts, among them J1 PI_CONN, J10 GND, J11 PSU_CONN, J12 3V3_PSU, J13 5V_PSU, J14 5V_SB, J15 12V_PSU, J16 POWER_GOOD, J17 PS_ON, J18 GND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

Commit message: Fixed board geometry to fit Raspberry Pi HAT spec better
Other:
- title: ATX-PSU-ProtoHAT-0010 -> ATX-PSU-ProtoHAT-0011
Changed lines of the file:
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@@
   (paper "A4")
   (title_block
-    (title "ATX-PSU-ProtoHAT-0010")
-    (date "2023-05-07")
+    (title "ATX-PSU-ProtoHAT-0011")
+    (date "2023-05-28")
     (rev "1.0")
     (company "(c) 2023 Andriy Golovnya")
